Commit message: feat: 更新URDF文件中的关节限制和轴方向

File: resources/robots/OpenDogV1.1/urdf/OpenDog.SLDASM.urdf (robot description, URDF)
Before this commit: robot OpenDog.SLDASM, 13 links, 12 joints
Joints:
- joint FL_calf_joint: axis 0 -1 0 -> 0 1 0; limit lower=0 upper=0 effort=0 velocity=0 -> lower=-2.68 upper=-1.04 effort=9 velocity=6.981
- joint FL_thigh_joint: limit lower=0 upper=0 effort=0 velocity=0 -> lower=-1.046799 upper=1.395799 effort=6 velocity=10.472
- joint FR_calf_joint: limit lower=0 upper=0 effort=0 velocity=0 -> lower=1.04 upper=2.68 effort=9 velocity=6.981
- joint FR_hip_joint: axis -1 0 0 -> 1 0 0; limit lower=0 upper=0 effort=0 velocity=0 -> lower=-0.521799 upper=1.046799 effort=6 velocity=10.472
- joint FR_thigh_joint: limit lower=0 upper=0 effort=0 velocity=0 -> lower=-1.395799 upper=1.046799 effort=6 velocity=10.472
- joint Fl_hip_joint: axis -1 0 0 -> 1 0 0; limit lower=0 upper=0 effort=0 velocity=0 -> lower=-1.046799 upper=0.521799 effort=6 velocity=10.472
- joint RL_calf_joint: axis 0 -1 0 -> 0 1 0; limit lower=0 upper=0 effort=0 velocity=0 -> lower=-2.68 upper=-1.04 effort=9 velocity=6.981
- joint RL_hip_joint: limit lower=0 upper=0 effort=0 velocity=0 -> lower=-0.521799 upper=1.046799 effort=6 velocity=10.472
- joint RL_thigh_joint: limit lower=0 upper=0 effort=0 velocity=0 -> lower=-1.046799 upper=1.395799 effort=6 velocity=10.472
- joint RR_calf_joint: axis 0 1 0 -> 0 -1 0; limit lower=0 upper=0 effort=0 velocity=0 -> lower=1.04 upper=2.68 effort=9 velocity=6.981
- joint RR_hip_joint: limit lower=0 upper=0 effort=0 velocity=0 -> lower=-1.046799 upper=0.521799 effort=6 velocity=10.472
- joint RR_thigh_joint: limit lower=0 upper=0 effort=0 velocity=0 -> lower=-1.395799 upper=1.046799 effort=6 velocity=10.472

Commit message: feat: 添加OpenDog V1.1支持，包括配置文件和训练任务

File: resources/robots/OpenDogV1.1/urdf/OpenDog.SLDASM.urdf (robot description, URDF)
Before this commit: robot OpenDog.SLDASM, 13 links, 12 joints
Links:
- removed link Fl_hip
- added link FL_hip, mass 0.2945; collision mesh filename=package://OpenDog.SLDASM/meshes/Fl_hip.STL; visual mesh filename=package://OpenDog.SLDASM/meshes/Fl_hip.STL
Joints:
- removed joint Fl_hip_joint
- added joint FL_hip_joint: type revolute, parent base_link, child FL_hip, origin xyz=0.095 0.04 0.002 rpy=0 0 0, axis 1 0 0, limit lower=-1.046799 upper=0.521799 effort=6 velocity=10.472
- joint FL_thigh_joint: parent Fl_hip -> FL_hip

Commit message: fix: 修正FL_hip模型文件名大小写以确保正确加载

File: resources/robots/OpenDogV1.1/urdf/OpenDog.SLDASM.urdf (robot description, URDF)
Before this commit: robot OpenDog.SLDASM, 13 links, 12 joints
Links:
- link FL_hip: geometry collision mesh filename=package://OpenDog.SLDASM/meshes/FL_hip.STL; visual mesh filename=package://OpenDog.SLDASM/meshes/FL_hip.STL

Commit message: feat: 更新OpenDog V1.1配置，添加前后脚链接和关节

File: resources/robots/OpenDogV1.1/urdf/OpenDog.SLDASM.urdf (robot description, URDF)
Before this commit: robot OpenDog.SLDASM, 13 links, 12 joints
Links:
- added link FL_foot, mass 0.001; collision sphere radius=0.015
- added link FR_foot, mass 0.001; collision sphere radius=0.015
- added link RL_foot, mass 0.001; collision sphere radius=0.015
- added link RR_foot, mass 0.001; collision sphere radius=0.015
Joints:
- added joint FL_foot_joint: type fixed, parent FL_calf, child FL_foot, origin xyz=0 0 -0.1 rpy=0 0 0
- added joint FR_foot_joint: type fixed, parent FR_calf, child FR_foot, origin xyz=0 0 -0.1 rpy=0 0 0
- added joint RL_foot_joint: type fixed, parent RL_calf, child RL_foot, origin xyz=0 0 -0.1 rpy=0 0 0
- added joint RR_foot_joint: type fixed, parent RR_calf, child RR_foot, origin xyz=0 0 -0.1 rpy=0 0 0
