Commit message: feat: 更新OpenDog V1.1配置，调整关节角度和文件路径

File: resources/robots/OpenDogV1.1/urdf/OpenDogV1_1.urdf (robot description, URDF)
Before this commit: robot OpenDog.SLDASM, 17 links, 16 joints
Links:
- link FL_calf: geometry collision mesh filename=../meshes/FL_calf.STL; visual mesh filename=../meshes/FL_calf.STL
- link FL_hip: geometry collision mesh filename=../meshes/FL_hip.STL; visual mesh filename=../meshes/FL_hip.STL
- link FL_thigh: geometry collision mesh filename=../meshes/FL_thigh.STL; visual mesh filename=../meshes/FL_thigh.STL
- link FR_calf: geometry collision mesh filename=../meshes/FR_calf.STL; visual mesh filename=../meshes/FR_calf.STL
- link FR_hip: geometry collision mesh filename=../meshes/FR_hip.STL; visual mesh filename=../meshes/FR_hip.STL
- link FR_thigh: geometry collision mesh filename=../meshes/FR_thigh.STL; visual mesh filename=../meshes/FR_thigh.STL
- link RL_calf: geometry collision mesh filename=../meshes/RL_calf.STL; visual mesh filename=../meshes/RL_calf.STL
- link RL_hip: geometry collision mesh filename=../meshes/RL_hip.STL; visual mesh filename=../meshes/RL_hip.STL
- link RL_thigh: geometry collision mesh filename=../meshes/RL_thigh.STL; visual mesh filename=../meshes/RL_thigh.STL
- link RR_calf: geometry collision mesh filename=../meshes/RR_calf.STL; visual mesh filename=../meshes/RR_calf.STL
- link RR_hip: geometry collision mesh filename=../meshes/RR_hip.STL; visual mesh filename=../meshes/RR_hip.STL
- link RR_thigh: geometry collision mesh filename=../meshes/RR_thigh.STL; visual mesh filename=../meshes/RR_thigh.STL
- link base_link: geometry collision mesh filename=../meshes/base_link.STL; visual mesh filename=../meshes/base_link.STL

Commit message: feat: 更新OpenDog V1.1配置，添加DOF重置噪声范围和关节速度限制

File: resources/robots/OpenDogV1.1/urdf/OpenDogV1_1.urdf (robot description, URDF)
Before this commit: robot OpenDog.SLDASM, 17 links, 16 joints
Links:
- link FL_calf: geometry collision box size=0.012 0.008 0.075; visual mesh filename=../meshes/FL_calf.STL
- link FL_hip: geometry collision cylinder length=0.055 radius=0.017; visual mesh filename=../meshes/FL_hip.STL
- link FL_thigh: geometry collision box size=0.018 0.014 0.055; collision cylinder length=0.035 radius=0.017
- link FR_calf: geometry collision box size=0.012 0.008 0.075; visual mesh filename=../meshes/FR_calf.STL
- link FR_hip: geometry collision cylinder length=0.050 radius=0.017; visual mesh filename=../meshes/FR_hip.STL
- link FR_thigh: geometry collision box size=0.018 0.014 0.055; collision cylinder length=0.035 radius=0.017
- link RL_calf: geometry collision box size=0.012 0.008 0.075; visual mesh filename=../meshes/RL_calf.STL
- link RL_hip: geometry collision cylinder length=0.050 radius=0.017; visual mesh filename=../meshes/RL_hip.STL
- link RL_thigh: geometry collision box size=0.018 0.014 0.055; collision cylinder length=0.035 radius=0.017
- link RR_calf: geometry collision box size=0.012 0.008 0.075; visual mesh filename=../meshes/RR_calf.STL
- link RR_hip: geometry collision cylinder length=0.050 radius=0.017; visual mesh filename=../meshes/RR_hip.STL
- link RR_thigh: geometry collision box size=0.018 0.014 0.055; collision cylinder length=0.035 radius=0.017
- link base_link: geometry collision box size=0.198 0.145 0.080; visual mesh filename=../meshes/base_link.STL
